File: src/hardware/hamdallv2.brd (EAGLE design)
At the start: 67 x 22.9 mm, 34 parts, among them IC1 MCP3008

Commit message: As sent to joe 7-27-2019
Parts:
- removed 1IN, 2IN, 4IN, 6IN, 7IN, 8IN: LSP11, solpad:LSP11
- added 1, 2, 4, 5, 7, 8: LSP11, solpad:LSP11
- moved HEADER 12.0 mm to (52.1, 61.0), turned to 180 degrees
- moved IC1 7.18 mm to (50.8, 69.8), turned to 180 degrees
- renumbered 1OUT to 1O, 2OUT to 2O, 3IN to 3, 3OUT to 3O, 4OUT to 4O, 5IN to 6, 5OUT to 5O, 6OUT to 6O, 7OUT to 7O, 8OUT to 8O
Connections:
- net PWR: now also 1.MP, 2.MP, 4.MP, 5.MP, 7.MP, 8.MP; no longer 1IN.MP, 2IN.MP, 4IN.MP, 6IN.MP, 7IN.MP, 8IN.MP
Routing:
- net GND: track 0.00 -> 108.6 mm
- net N$9: track 0.00 -> 57.8 mm
- net N$2: track 0.00 -> 57.2 mm
- net N$3: track 0.00 -> 54.6 mm
- net N$6: track 0.00 -> 54.6 mm
- net N$5: track 0.00 -> 54.6 mm
- net N$4: track 0.00 -> 53.7 mm
- net N$7: track 0.00 -> 48.4 mm
- net N$8: track 0.00 -> 46.3 mm
- net PWR: track 0.00 -> 37.4 mm
- net N$11: track 0.00 -> 5.61 mm
- net N$14: track 0.00 -> 5.61 mm
- net N$13: track 0.00 -> 5.61 mm
- net N$12: track 0.00 -> 5.61 mm
Other:
- board size 67 x 22.9 mm -> 63.2 x 22.9 mm
- board text added: "IN"

Commit message: As ordered 7-27-2019
Parts:
- moved 1 1.27 mm to (39.4, 77.5)
- moved 2 1.27 mm to (41.9, 77.5)
- moved 6 1.27 mm to (52.1, 77.5)
- moved 7 1.27 mm to (54.6, 77.5)
- moved 8 1.27 mm to (57.1, 77.5)
- moved IC1 1.27 mm to (52.1, 69.8)
- moved 4O 1.27 mm to (16.5, 77.5)
- moved 2O 1.27 mm to (8.89, 77.5)
- moved 1O 1.27 mm to (5.08, 77.5)
- moved 3O 1.27 mm to (12.7, 77.5)
- moved 5O 1.27 mm to (20.3, 77.5)
- moved 6O 1.27 mm to (24.1, 77.5)
- moved 7O 1.27 mm to (27.9, 77.5)
- moved 8O 1.27 mm to (31.8, 77.5)
- moved 3 1.27 mm to (44.5, 77.5)
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Routing:
- net N$3: track 54.6 -> 49.0 mm
- net N$9: track 57.8 -> 52.3 mm
- net GND: track 108.6 -> 105.1 mm
- net N$6: track 54.6 -> 51.5 mm
- net N$5: track 54.6 -> 52.8 mm
- net PWR: track 37.4 -> 38.8 mm
- net N$7: track 48.4 -> 49.8 mm
- net N$14: track 5.61 -> 5.08 mm
- net N$12: track 5.61 -> 5.08 mm
